File: PCB/HomeEnvSensor/HomeEnvSensor.kicad_pcb (KiCad board)
At the start: 2 copper layers, 1 part, among them U1 STM32L031F6P7

Commit message: udated by FZ from Windows
Parts:
- added C1: 0.1uF, Capacitor_SMD:C_0402_1005Metric_Pad0.74x0.62mm_HandSolder, F.Cu at (165.2, 97.0)
- added C10: 22pF, Capacitor_SMD:C_0402_1005Metric_Pad0.74x0.62mm_HandSolder, F.Cu at (165.2, 101.0)
- added C2: 10uF, Capacitor_SMD:C_0603_1608Metric_Pad1.08x0.95mm_HandSolder, F.Cu at (133.4, 106.8)
- added C3: 0.01uF, Capacitor_SMD:C_0402_1005Metric_Pad0.74x0.62mm_HandSolder, F.Cu at (145.9, 106.5)
- added C4: 0.1uF, Capacitor_SMD:C_0402_1005Metric_Pad0.74x0.62mm_HandSolder, F.Cu at (145.9, 108.5)
- added C5: 4.7uF, Capacitor_SMD:C_0603_1608Metric_Pad1.08x0.95mm_HandSolder, F.Cu at (133.4, 109.3)
- added C6: 0.1uF, Capacitor_SMD:C_0402_1005Metric_Pad0.74x0.62mm_HandSolder, F.Cu at (145.9, 110.5)
- added C7: 4.7uF, Capacitor_SMD:C_0603_1608Metric_Pad1.08x0.95mm_HandSolder, F.Cu at (133.4, 111.8)
- added C8: 22uF, Capacitor_SMD:C_0805_2012Metric_Pad1.18x1.45mm_HandSolder, F.Cu at (146.2, 124.0)
- added C9: 22pF, Capacitor_SMD:C_0402_1005Metric_Pad0.74x0.62mm_HandSolder, F.Cu at (165.2, 99.0)
- added D1: RED, LED_SMD:LED_0603_1608Metric_Pad1.05x0.95mm_HandSolder, F.Cu at (141.0, 124.4)
- added J1: USB_B_Micro, Connector_USB:USB_Micro-B_Amphenol_10104110_Horizontal, F.Cu at (160.6, 134.3)
- added J4: Battery, Connector_PinHeader_2.00mm:PinHeader_1x02_P2.00mm_Vertical, F.Cu at (151.8, 101.4)
- added L1: 22uH, Inductor_SMD:L_Taiyo-Yuden_NR-40xx_HandSoldering, F.Cu at (135.0, 120.9)
- added L2: 4.7uH, Inductor_SMD:L_Wuerth_MAPI-3015, F.Cu at (141.3, 120.6)
- added R1: 0, Resistor_SMD:R_0603_1608Metric_Pad0.98x0.95mm_HandSolder, F.Cu at (133.4, 114.3)
- added R10: 8.25M, Resistor_SMD:R_0603_1608Metric_Pad0.98x0.95mm_HandSolder, F.Cu at (142.1, 111.8)
- added R11: 4.75M, Resistor_SMD:R_0603_1608Metric_Pad0.98x0.95mm_HandSolder, F.Cu at (142.1, 114.3)
- added R12: 499k, Resistor_SMD:R_0603_1608Metric_Pad0.98x0.95mm_HandSolder, F.Cu at (133.4, 129.0)
- added R13: 499k, Resistor_SMD:R_0603_1608Metric_Pad0.98x0.95mm_HandSolder, F.Cu at (133.4, 131.5)
- added R14: 499k, Resistor_SMD:R_0603_1608Metric_Pad0.98x0.95mm_HandSolder, F.Cu at (133.4, 134.0)
- added R15: 499k, Resistor_SMD:R_0603_1608Metric_Pad0.98x0.95mm_HandSolder, F.Cu at (133.4, 136.5)
- added R16: 4.7K, Resistor_SMD:R_0603_1608Metric_Pad0.98x0.95mm_HandSolder, F.Cu at (169.0, 97.3)
- added R17: 4.7K, Resistor_SMD:R_0603_1608Metric_Pad0.98x0.95mm_HandSolder, F.Cu at (169.0, 99.8)
- added R2: 10k, Resistor_SMD:R_0603_1608Metric_Pad0.98x0.95mm_HandSolder, F.Cu at (133.4, 116.8)
- added R3: 100, Resistor_SMD:R_0603_1608Metric_Pad0.98x0.95mm_HandSolder, F.Cu at (137.8, 106.8)
- added R4: 7.32M, Resistor_SMD:R_0603_1608Metric_Pad0.98x0.95mm_HandSolder, F.Cu at (137.8, 109.3)
- added R5: 5.62M, Resistor_SMD:R_0603_1608Metric_Pad0.98x0.95mm_HandSolder, F.Cu at (137.8, 111.8)
- added R6: 330K, Resistor_SMD:R_0603_1608Metric_Pad0.98x0.95mm_HandSolder, F.Cu at (137.8, 114.3)
- added R7: 8.45M, Resistor_SMD:R_0603_1608Metric_Pad0.98x0.95mm_HandSolder, F.Cu at (137.8, 116.8)
- added R8: 4.22M, Resistor_SMD:R_0603_1608Metric_Pad0.98x0.95mm_HandSolder, F.Cu at (142.1, 106.8)
- added R9: 10k, Resistor_SMD:R_0603_1608Metric_Pad0.98x0.95mm_HandSolder, F.Cu at (142.1, 109.3)
- added U3: BQ25570, Package_DFN_QFN:QFN-20-1EP_3.5x3.5mm_P0.5mm_EP2x2mm, F.Cu at (161.3, 108.2)
- added U4: MCP73831-2-OT, Package_TO_SOT_SMD:SOT-23-5, F.Cu at (174.0, 106.4)
- added Y1: 32.768KHz, Crystal:Crystal_SMD_0603-2Pin_6.0x3.5mm_HandSoldering, F.Cu at (152.4, 117.7)
- moved U1 36.3 mm to (161.7, 119.0)
Connections:
- net /BOOT renamed BOOT
- net /SWDCLK renamed SWDCLK
- net /SWDIO renamed SWDIO
- net /~{RST} renamed ~{RST}
- U1 pad 10: unconnected-(U1-PA4-Pad10) -> NSS
- U1 pad 11: unconnected-(U1-PA5-Pad11) -> SCK
- U1 pad 12: unconnected-(U1-PA6-Pad12) -> MISO
- U1 pad 13: unconnected-(U1-PA7-Pad13) -> MOSI
- U1 pad 14: unconnected-(U1-PB1-Pad14) -> LED
- U1 pad 17: unconnected-(U1-PA9-Pad17) -> SCL
- U1 pad 18: unconnected-(U1-PA10-Pad18) -> SDA
- U1 pad 2: /OSC_32_in -> Net-(U1-PC14)
- U1 pad 3: /OSC_32_out -> Net-(U1-PC15)
- U1 pad 6: unconnected-(U1-PA0-Pad6) -> ADC_IN0
- U1 pad 7: unconnected-(U1-PA1-Pad7) -> ADC_IN1
- U1 pad 8: unconnected-(U1-PA2-Pad8) -> USER_IN
- U1 pad 9: unconnected-(U1-PA3-Pad9) -> USER_OUT
