File: PCB/HomeEnvSensor/HomeEnvSensor.kicad_sch (KiCad schematic)
At the start: 3 parts, among them J1 Connector, U1 STM32L031F6P7

Commit message: udated by FZ from Windows
Parts:
- removed C1: C_Small, symbol Device:C_Small
- removed J1: Connector, symbol Connector:Conn_01x06_Pin
- removed U1: STM32L031F6P7, Package_SO:TSSOP-20_4.4x6.5mm_P0.65mm, symbol MCU_ST_STM32L0:STM32L031F6Px
Other:
- added sheet Conn (Conn.kicad_sch)
- added sheet MCU (MCU.kicad_sch)
- added sheet Power (Power.kicad_sch)
